File: EAGLE Files/ACT Lipoly Charger R3 FINAL.sch (EAGLE design)
At the start: 150 parts, among them J12 Bk, J13 Sel, J14 Fwd, U1 74HC595

Commit message: Adds missing LCD signal traces
Connections:
- net D2: now also J15.6
- net D3: now also J15.5
- net D4: now also J15.4
- net D5: now also J15.3
- net GND: now also J15.1
- net VCC: now also J15.2
Changed lines of the file:
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@@
 <?xml version="1.0" encoding="utf-8"?>
 <!DOCTYPE eagle SYSTEM "eagle.dtd">
-<eagle version="7.6.0">
+<eagle version="8.2.2">
 <drawing>
 <settings>
@@
 </segment>
 <segment>
-<wire x1="-109.22" y1="121.92" x2="-106.68" y2="121.92" width="0.1524" layer="91"/>
-<label x="-106.68" y="121.92" size="1.778" layer="95"/>
-</segment>
-<segment>
 <wire x1="-109.22" y1="149.86" x2="-106.68" y2="149.86" width="0.1524" layer="91"/>
 <label x="-106.68" y="149.86" size="1.778" layer="95"/>
@@
 <wire x1="-160.02" y1="78.74" x2="-157.48" y2="78.74" width="0.1524" layer="91"/>
 <label x="-157.48" y="78.74" size="1.778" layer="95"/>
+</segment>
+<segment>
+<pinref part="J15" gate="G$1" pin="1"/>
+<wire x1="-109.22" y1="121.92" x2="-106.68" y2="121.92" width="0.1524" layer="91"/>
+<label x="-106.68" y="121.92" size="1.778" layer="95"/>
 </segment>
 </net>
@@
 <junction x="228.6" y="-88.9"/>
 <pinref part="SUPPLY15" gate="G$1" pin="VCC"/>
-</segment>
-<segment>
-<wire x1="-109.22" y1="124.46" x2="-106.68" y2="124.46" width="0.1524" layer="91"/>
-<label x="-106.68" y="124.46" size="1.778" layer="95"/>
 </segment>
 <segment>
@@
 <wire x1="76.2" y1="-10.16" x2="81.28" y2="-10.16" width="0.1524" layer="91"/>
 <junction x="76.2" y="-10.16"/>
+</segment>
+<segment>
+<pinref part="J15" gate="G$1" pin="2"/>
+<wire x1="-109.22" y1="124.46" x2="-106.68" y2="124.46" width="0.1524" layer="91"/>
+<label x="-106.68" y="124.46" size="1.778" layer="95"/>
 </segment>
 </net>
@@
 </segment>
 <segment>
+<pinref part="J15" gate="G$1" pin="3"/>
 <wire x1="-109.22" y1="127" x2="-106.68" y2="127" width="0.1524" layer="91"/>
 <label x="-106.68" y="127" size="1.778" layer="95"/>
@@
 </segment>
 <segment>
+<pinref part="J15" gate="G$1" pin="4"/>
 <wire x1="-109.22" y1="129.54" x2="-106.68" y2="129.54" width="0.1524" layer="91"/>
 <label x="-106.68" y="129.54" size="1.778" layer="95"/>
@@
 </segment>
 <segment>
+<pinref part="J15" gate="G$1" pin="5"/>
 <wire x1="-109.22" y1="132.08" x2="-106.68" y2="132.08" width="0.1524" layer="91"/>
 <label x="-106.68" y="132.08" size="1.778" layer="95"/>
@@
 </segment>
 <segment>
+<pinref part="J15" gate="G$1" pin="6"/>
 <wire x1="-109.22" y1="134.62" x2="-106.68" y2="134.62" width="0.1524" layer="91"/>
 <label x="-106.68" y="134.62" size="1.778" layer="95"/>
